Commit message: able to visualize UR5e arm in drake

File: ur5e.urdf (robot description, URDF)
Before this commit: robot ur5e, 13 links, 12 joints
Links:
- link base_link_inertia: geometry collision mesh filename=./meshes/ur5e/collision/base.obj; visual mesh filename=./meshes/ur5e/visual/base.obj
- link forearm_link: geometry collision mesh filename=./meshes/ur5e/collision/forearm.obj; visual mesh filename=./meshes/ur5e/visual/forearm.obj
- link shoulder_link: geometry collision mesh filename=./meshes/ur5e/collision/shoulder.obj; visual mesh filename=./meshes/ur5e/visual/shoulder.obj
- link upper_arm_link: geometry collision mesh filename=./meshes/ur5e/collision/upperarm.obj; visual mesh filename=./meshes/ur5e/visual/upperarm.obj
- link wrist_1_link: geometry collision mesh filename=./meshes/ur5e/collision/wrist1.obj; visual mesh filename=./meshes/ur5e/visual/wrist1.obj
- link wrist_2_link: geometry collision mesh filename=./meshes/ur5e/collision/wrist2.obj; visual mesh filename=./meshes/ur5e/visual/wrist2.obj
- link wrist_3_link: geometry collision mesh filename=./meshes/ur5e/collision/wrist3.obj; visual mesh filename=./meshes/ur5e/visual/wrist3.obj
